Commit message: Updating RViz file launch.

File: src/pioneer_description/models/robots/pioneer.urdf (robot description, URDF)
Before this commit: robot pioneer3at_body, 19 links, 18 joints
Links:
- link chassis: geometry collision mesh filename=package://pioneer_description/meshes/chassis.dae; visual mesh filename=package://pioneer_description/meshes/chassis.dae
- link laser_frame: geometry collision box size=0.01 0.01 0.01; visual mesh filename=package://pioneer_description/meshes/hokuyo1.dae
- link p3at_back_left_axle: geometry collision box size=0.01 0.01 0.01; visual mesh filename=package://pioneer_description/meshes/p3at_meshes/axle.dae
- link p3at_back_left_hub: geometry collision box size=0.01 0.01 0.01; visual mesh filename=package://pioneer_description/meshes/p3at_meshes/left_hubca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
- link p3at_back_left_wheel: geometry collision mesh filename=package://pioneer_description/meshes/p3at_meshes/wheel.dae; visual mesh filename=package://pioneer_description/meshes/p3at_meshes/wheel.dae
- link p3at_back_right_axle: geometry collision box size=0.01 0.01 0.01; visual mesh filename=package://pioneer_description/meshes/p3at_meshes/axle.dae
- link p3at_back_right_hub: geometry collision box size=0.01 0.01 0.01; visual mesh filename=package://pioneer_description/meshes/p3at_meshes/right_hubc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
- link p3at_back_right_wheel: geometry collision mesh filename=package://pioneer_description/meshes/p3at_meshes/wheel.dae; visual mesh filename=package://pioneer_description/meshes/p3at_meshes/wheel.dae
- link p3at_front_left_axle: geometry collision box size=0.01 0.01 0.01; visual mesh filename=package://pioneer_description/meshes/p3at_meshes/axle.dae
- link p3at_front_left_hub: geometry collision box size=0.01 0.01 0.01; visual mesh filename=package://pioneer_description/meshes/p3at_meshes/left_hubca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
- link p3at_front_left_wheel: geometry collision mesh filename=package://pioneer_description/meshes/p3at_meshes/wheel.dae; visual mesh filename=package://pioneer_description/meshes/p3at_meshes/wheel.dae
- link p3at_front_right_axle: geometry collision box size=0.01 0.01 0.01; visual mesh filename=package://pioneer_description/meshes/p3at_meshes/axle.dae
- link p3at_front_right_hub: geometry collision box size=0.01 0.01 0.01; visual mesh filename=package://pioneer_description/meshes/p3at_meshes/right_hubc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
- link p3at_front_right_wheel: geometry collision mesh filename=package://pioneer_description/meshes/p3at_meshes/wheel.dae; visual mesh filename=package://pioneer_description/meshes/p3at_meshes/wheel.dae
- link top_plate: geometry collision box size=0.1 0.1 0.1; visual mesh filename=package://pioneer_description/meshes/top.dae

Commit message: Updating URDF file.

File: src/pioneer_description/models/robots/pioneer.urdf (robot description, URDF)
Before this commit: robot pioneer, 19 links, 18 joints
Links:
- removed link laser_frame
- added link cloud, mass 1e-5; collision box size=0.01 0.01 0.01; visual mesh filename=package://pioneer_description/meshes/hokuyo1.dae
Joints:
- joint laser_joint: child laser_frame -> cloud

Commit message: Addign EKF node.

File: src/pioneer_description/models/robots/pioneer.urdf (robot description, URDF)
Before this commit: robot pioneer, 19 links, 18 joints
Links:
- removed link cam_frame
- added link oak; visual box size=0.01 0.05 0.01
Joints:
- joint cam_joint: child cam_frame -> oak
- joint cam_optical_joint: parent cam_frame -> oak

Commit message: Update files.

File: src/pioneer_description/models/robots/pioneer.urdf (robot description, URDF)
Before this commit: robot pioneer, 19 links, 18 joints
Links:
- added link imu_link
Joints:
- added joint imu_joint: type fixed, parent base_link, child imu_link, origin xyz=0.24 0 0.271 rpy=0 0 0

Commit message: Update camera_tf launch file.

File: src/pioneer_description/models/robots/pioneer.urdf (robot description, URDF)
Before this commit: robot pioneer, 20 links, 19 joints
Links:
- removed link oak
- added link cam_link; visual box size=0.01 0.05 0.01
Joints:
- joint cam_joint: child oak -> cam_link
- joint cam_optical_joint: parent oak -> cam_link

Commit message: Robot description parameter.

File: src/pioneer_description/models/robots/pioneer.urdf (robot description, URDF)
Before this commit: robot pioneer, 20 links, 19 joints
Joints:
- joint p3at_back_left_wheel_joint: type continuous -> fixed
- joint p3at_back_right_wheel_joint: type continuous -> fixed
- joint p3at_front_left_wheel_joint: type continuous -> fixed
- joint p3at_front_right_wheel_joint: type continuous -> fixed
