Commit message: Simulation.

File: src/pioneer_description/models/robots/backup.urdf (robot description, URDF)
Before this commit: robot pioneer3at_body, 19 links, 18 joints
Links:
- removed link cam_frame
- removed link laser_frame
- added link cam_link; visual box size=0.01 0.05 0.01
- added link cloud, mass 1e-5; collision box size=0.01 0.01 0.01; visual mesh filename=package://pioneer_description/meshes/hokuyo1.dae
- added link imu_link
- link chassis: geometry collision mesh filename=package://pioneer_description/meshes/chassis.dae; visual mesh filename=package://pioneer_description/meshes/chassis.dae
- link p3at_back_left_axle: geometry collision box size=0.01 0.01 0.01; visual mesh filename=package://pioneer_description/meshes/p3at_meshes/axle.dae
- link p3at_back_left_hub: geometry collision box size=0.01 0.01 0.01; visual mesh filename=package://pioneer_description/meshes/p3at_meshes/left_hubca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
- link p3at_back_left_wheel: geometry collision mesh filename=package://pioneer_description/meshes/p3at_meshes/wheel.dae; visual mesh filename=package://pioneer_description/meshes/p3at_meshes/wheel.dae
- link p3at_back_right_axle: geometry collision box size=0.01 0.01 0.01; visual mesh filename=package://pioneer_description/meshes/p3at_meshes/axle.dae
- link p3at_back_right_hub: geometry collision box size=0.01 0.01 0.01; visual mesh filename=package://pioneer_description/meshes/p3at_meshes/right_hubc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
- link p3at_back_right_wheel: geometry collision mesh filename=package://pioneer_description/meshes/p3at_meshes/wheel.dae; visual mesh filename=package://pioneer_description/meshes/p3at_meshes/wheel.dae
- link p3at_front_left_axle: geometry collision box size=0.01 0.01 0.01; visual mesh filename=package://pioneer_description/meshes/p3at_meshes/axle.dae
- link p3at_front_left_hub: geometry collision box size=0.01 0.01 0.01; visual mesh filename=package://pioneer_description/meshes/p3at_meshes/left_hubca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
- link p3at_front_left_wheel: geometry collision mesh filename=package://pioneer_description/meshes/p3at_meshes/wheel.dae; visual mesh filename=package://pioneer_description/meshes/p3at_meshes/wheel.dae
- link p3at_front_right_axle: geometry collision box size=0.01 0.01 0.01; visual mesh filename=package://pioneer_description/meshes/p3at_meshes/axle.dae
- link p3at_front_right_hub: geometry collision box size=0.01 0.01 0.01; visual mesh filename=package://pioneer_description/meshes/p3at_meshes/right_hubc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
- link p3at_front_right_wheel: geometry collision mesh filename=package://pioneer_description/meshes/p3at_meshes/wheel.dae; visual mesh filename=package://pioneer_description/meshes/p3at_meshes/wheel.dae
- link top_plate: geometry collision box size=0.1 0.1 0.1; visual mesh filename=package://pioneer_description/meshes/top.dae
Joints:
- added joint imu_joint: type fixed, parent base_link, child imu_link, origin xyz=0.24 0 0.271 rpy=0 0 0
- joint cam_joint: child cam_frame -> cam_link
- joint cam_optical_joint: parent cam_frame -> cam_link
- joint laser_joint: child laser_frame -> cloud
- joint p3at_back_left_wheel_joint: type continuous -> fixed
- joint p3at_back_right_wheel_joint: type continuous -> fixed
- joint p3at_front_left_wheel_joint: type continuous -> fixed
- joint p3at_front_right_wheel_joint: type continuous -> fixed
